File: 6502Kicad/6502Kicad.sch (KiCad schematic (older format))
At the start: 6 parts, among them SW1 SW_Push, U1 W65C02S

Commit message: changed push button lib to correctly linked lib
Parts:
- removed U1: W65C02S, Package_DIP:DIP-40_W15.24mm_Socket, symbol 6502:W65C02S
- added U?: W65C02S, symbol 6502:W65C02S
- SW1: symbol tmc:SW_Push -> 6502:SW_Push
Connections:
- net +3V3: now also U?.36 (BE), U?.6 (NMI), U?.8 (VDD)
- net A0: now also U?.9 (A0)
- net A1: now also U?.10 (A1)
- net A10: now also U?.19 (A10)
- net A11: now also U?.20 (A11)
- net A12: now also U?.22 (A12)
- net A13: now also U?.23 (A13)
- net A14: now also U?.24 (A14)
- net A15: now also U?.25 (A15)
- net A2: now also U?.11 (A2)
- net A3: now also U?.12 (A3)
- net A4: now also U?.13 (A4)
- net A5: now also U?.14 (A5)
- net A6: now also U?.15 (A6)
- net A7: now also U?.16 (A7)
- net A8: now also U?.17 (A8)
- net A9: now also U?.18 (A9)
- net BusR~W~: now also U?.34 (R/~W~)
- net Clk: now also U?.37 (PHI2)
- net D0: now also U?.33 (D0)
- net D1: now also U?.32 (D1)
- net D2: now also U?.31 (D2)
- net D3: now also U?.30 (D3)
- net D4: now also U?.29 (D4)
- net D5: now also U?.28 (D5)
- net D6: now also U?.27 (D6)
- net D7: now also U?.26 (D7)
- net GND: now also U?.21 (VSS)
- net ~IRQ: now also U?.4 (IRQ)
- net at R2.1: now also U?.2 (RDY)
- net at C1.1, R1.1, SW1.2: now also U?.40 (RST)
Changed lines of the file:
@@
-	1    0    0    -1
-$EndComp
-$Comp
-L 6502:W65C02S U1
-U 1 1 61ECFD65
-P 2000 2300
-F 0 "U1" H 2150 3600 50  0000 C CNN
-F 1 "W65C02S" H 1750 3600 50  0000 C CNN
-F 2 "Package_DIP:DIP-40_W15.24mm_Socket" H 2100 3600 50  0001 C CNN
-F 3 "" H 2100 3600 50  0001 C CNN
-	1    2000 2300
 	1    0    0    -1
 $EndComp
@@
 	1500 1650 1350 1650
 $Comp
-L tmc:SW_Push SW1
+L 6502:SW_Push SW1
 U 1 1 61EDE944
 P 1350 1850
@@
 Text Label 1300 1350 0    50   ~ 0
 ~IRQ
+$Comp
+L 6502:W65C02S U?
+U 1 1 61ECCCF2
+P 2000 2300
+F 0 "U?" H 1700 3600 50  0000 C CNN
+F 1 "W65C02S" H 2200 3600 50  0000 C CNN
+F 2 "" H 2100 3600 50  0001 C CNN
+F 3 "" H 2100 3600 50  0001 C CNN
+	1    2000 2300
+	1    0    0    -1
+$EndComp
+$Comp
+L power:GND #PWR?
+U 1 1 61ECFC82
+P 2000 3750
+F 0 "#PWR?" H 2000 3500 50  0001 C CNN
+F 1 "GND" H 2005 3577 50  0000 C CNN
+F 2 "" H 2000 3750 50  0001 C CNN
+F 3 "" H 2000 3750 50  0001 C CNN
+	1    2000 3750
+	1    0    0    -1
+$EndComp
+Wire Wire Line
+	2000 3750 2000 3700
 Wire Bus Line
 	2950 1150 2950 3450
